File: basspreamp.sch (KiCad schematic (older format))
At the start: 27 parts, among them P1 INPUT, P2 OUTPUT, P3 Power, Q1 J201, U1 TL072

Commit message: Add filled zone to pcb, make prints
Parts:
- U1: symbol TL072 -> TL072-RESCUE-basspreamp
Changed lines of the file:
@@
 EESchema Schematic File Version 2
+LIBS:basspreamp-rescue
 LIBS:power
 LIBS:device
@@
 Connection ~ 4100 2900
 $Comp
-L TL072 U1
+L TL072-RESCUE-basspreamp U1
 U 1 1 561CCF45
 P 5100 3000
@@
 Connection ~ 5600 3800
 $Comp
-L TL072 U1
+L TL072-RESCUE-basspreamp U1
 U 2 1 561CE4B3
 P 8250 4100
